Commit message: Update URDF with imu

File: thunder_description/urdf/thunder.xacro (robot description, xacro)
@@ -6,7 +6,7 @@
 <link name="base_link">
   <inertial>
-    <origin xyz="-0.001413748491849484 -7.829515970253678e-07 0.06686697168936584" rpy="0 0 0"/>
-    <mass value="2.30327736288842"/>
-    <inertia ixx="0.006108" iyy="0.010564" izz="0.008297" ixy="0.0" iyz="-0.0" ixz="0.000265"/>
+    <origin xyz="-0.0015343514816687786 -7.81885672034026e-07 0.06692160954933128" rpy="0 0 0"/>
+    <mass value="2.306417362888421"/>
+    <inertia ixx="0.006113" iyy="0.010594" izz="0.008322" ixy="0.0" iyz="-0.0" ixz="0.000276"/>
   </inertial>
   <visual>
@@ -24,5 +24,5 @@
   </collision>
 </link>
-<link name="left_wheel_front_1">
+<link name="front_wheel_left_1">
   <inertial>
     <origin xyz="-1.3877787807814457e-17 0.012500000000000004 0.0" rpy="0 0 0"/>
@@ -33,5 +33,5 @@
     <origin xyz="-0.07 -0.043 -0.0325" rpy="0 0 0"/>
     <geometry>
-      <mesh filename="file://$(find thunder_description)/meshes/left_wheel_front_1.stl" scale="0.001 0.001 0.001"/>
+      <mesh filename="file://$(find thunder_description)/meshes/front_wheel_left_1.stl" scale="0.001 0.001 0.001"/>
     </geometry>
     <material name="silver"/>
@@ -40,9 +40,9 @@
     <origin xyz="-0.07 -0.043 -0.0325" rpy="0 0 0"/>
     <geometry>
-      <mesh filename="file://$(find thunder_description)/meshes/left_wheel_front_1.stl" scale="0.001 0.001 0.001"/>
-    </geometry>
-  </collision>
-</link>
-<link name="right_wheel_front_1">
+      <mesh filename="file://$(find thunder_description)/meshes/front_wheel_left_1.stl" scale="0.001 0.001 0.001"/>
+    </geometry>
+  </collision>
+</link>
+<link name="front_wheel_right_1">
   <inertial>
     <origin xyz="0.0 -0.012500000000000004 0.0" rpy="0 0 0"/>
@@ -53,5 +53,5 @@
     <origin xyz="-0.07 0.043 -0.0325" rpy="0 0 0"/>
     <geometry>
-      <mesh filename="file://$(find thunder_description)/meshes/right_wheel_front_1.stl" scale="0.001 0.001 0.001"/>
+      <mesh filename="file://$(find thunder_description)/meshes/front_wheel_right_1.stl" scale="0.001 0.001 0.001"/>
     </geometry>
     <material name="silver"/>
@@ -60,9 +60,9 @@
     <origin xyz="-0.07 0.043 -0.0325" rpy="0 0 0"/>
     <geometry>
-      <mesh filename="file://$(find thunder_description)/meshes/right_wheel_front_1.stl" scale="0.001 0.001 0.001"/>
-    </geometry>
-  </collision>
-</link>
-<link name="left_wheel_rear_1">
+      <mesh filename="file://$(find thunder_description)/meshes/front_wheel_right_1.stl" scale="0.001 0.001 0.001"/>
+    </geometry>
+  </collision>
+</link>
+<link name="rear_wheel_left_1">
   <inertial>
     <origin xyz="2.7755575615628914e-17 0.012500000000000004 0.0" rpy="0 0 0"/>
@@ -73,5 +73,5 @@
     <origin xyz="0.07 -0.043 -0.0325" rpy="0 0 0"/>
     <geometry>
-      <mesh filename="file://$(find thunder_description)/meshes/left_wheel_rear_1.stl" scale="0.001 0.001 0.001"/>
+      <mesh filename="file://$(find thunder_description)/meshes/rear_wheel_left_1.stl" scale="0.001 0.001 0.001"/>
     </geometry>
     <material name="silver"/>
@@ -80,9 +80,9 @@
     <origin xyz="0.07 -0.043 -0.0325" rpy="0 0 0"/>
     <geometry>
-      <mesh filename="file://$(find thunder_description)/meshes/left_wheel_rear_1.stl" scale="0.001 0.001 0.001"/>
-    </geometry>
-  </collision>
-</link>
-<link name="right_wheel_rear_1">
+      <mesh filename="file://$(find thunder_description)/meshes/rear_wheel_left_1.stl" scale="0.001 0.001 0.001"/>
+    </geometry>
+  </collision>
+</link>
+<link name="rear_wheel_right_1">
   <inertial>
     <origin xyz="1.3877787807814457e-17 -0.012500000000000004 0.0" rpy="0 0 0"/>
@@ -93,5 +93,5 @@
     <origin xyz="0.07 0.043 -0.0325" rpy="0 0 0"/>
     <geometry>
-      <mesh filename="file://$(find thunder_description)/meshes/right_wheel_rear_1.stl" scale="0.001 0.001 0.001"/>
+      <mesh filename="file://$(find thunder_description)/meshes/rear_wheel_right_1.stl" scale="0.001 0.001 0.001"/>
     </geometry>
     <material name="silver"/>
@@ -100,5 +100,5 @@
     <origin xyz="0.07 0.043 -0.0325" rpy="0 0 0"/>
     <geometry>
-      <mesh filename="file://$(find thunder_description)/meshes/right_wheel_rear_1.stl" scale="0.001 0.001 0.001"/>
+      <mesh filename="file://$(find thunder_description)/meshes/rear_wheel_right_1.stl" scale="0.001 0.001 0.001"/>
     </geometry>
   </collision>
@@ -144,26 +144,46 @@
   </collision>
 </link>
-<joint name="left_wheel_front_joint" type="continuous">
+<link name="imu_1">
+  <inertial>
+    <origin xyz="0.0 0.0 0.0010000000000000009" rpy="0 0 0"/>
+    <mass value="0.0062799999999999774"/>
+    <inertia ixx="0.0" iyy="0.0" izz="0.0" ixy="0.0" iyz="0.0" ixz="-0.0"/>
+  </inertial>
+  <visual>
+    <origin xyz="0.09 -0.0 -0.1075" rpy="0 0 0"/>
+    <geometry>
+      <mesh filename="file://$(find thunder_description)/meshes/imu_1.stl" scale="0.001 0.001 0.001"/>
+    </geometry>
+    <material name="silver"/>
+  </visual>
+  <collision>
+    <origin xyz="0.09 -0.0 -0.1075" rpy="0 0 0"/>
+    <geometry>
+      <mesh filename="file://$(find thunder_description)/meshes/imu_1.stl" scale="0.001 0.001 0.001"/>
+    </geometry>
+  </collision>
+</link>
+<joint name="front_wheel_left_joint" type="continuous">
   <origin xyz="0.07 0.043 0.0325" rpy="0 0 0"/>
   <parent link="base_link"/>
-  <child link="left_wheel_front_1"/>
+  <child link="front_wheel_left_1"/>
   <axis xyz="0.0 1.0 0.0"/>
 </joint>
-<joint name="right_wheel_front_joint" type="continuous">
+<joint name="front_wheel_right_joint" type="continuous">
   <origin xyz="0.07 -0.043 0.0325" rpy="0 0 0"/>
   <parent link="base_link"/>
-  <child link="right_wheel_front_1"/>
+  <child link="front_wheel_right_1"/>
   <axis xyz="0.0 -1.0 0.0"/>
 </joint>
-<joint name="left_wheel_rear_joint" type="continuous">
+<joint name="rear_wheel_left_joint" type="continuous">
   <origin xyz="-0.07 0.043 0.0325" rpy="0 0 0"/>
   <parent link="base_link"/>
-  <child link="left_wheel_rear_1"/>
+  <child link="rear_wheel_left_1"/>
   <axis xyz="0.0 1.0 0.0"/>
 </joint>
-<joint name="right_wheel_rear_joint" type="continuous">
+<joint name="rear_wheel_right_joint" type="continuous">
   <origin xyz="-0.07 -0.043 0.0325" rpy="0 0 0"/>
   <parent link="base_link"/>
-  <child link="right_wheel_rear_1"/>
+  <child link="rear_wheel_right_1"/>
   <axis xyz="0.0 -1.0 0.0"/>
 </joint>
@@ -173,8 +193,13 @@
   <child link="lidar_1"/>
 </joint>
-<joint name="camera_joint" type="fixed">
+<joint name="camera_link" type="fixed">
   <origin xyz="0.095 0.0 0.1075" rpy="0 0 0"/>
   <parent link="base_link"/>
   <child link="camera_1"/>
 </joint>
+<joint name="imu_link" type="fixed">
+  <origin xyz="-0.09 0.0 0.1075" rpy="0 0 0"/>
+  <parent link="base_link"/>
+  <child link="imu_1"/>
+</joint>
 </robot>

Commit message: Update Description

File: thunder_description/urdf/thunder.xacro (robot description, xacro)
@@ -24,5 +24,5 @@
   </collision>
 </link>
-<link name="front_wheel_left_1">
+<link name="front_wheel_left">
   <inertial>
     <origin xyz="-1.3877787807814457e-17 0.012500000000000004 0.0" rpy="0 0 0"/>
@@ -33,5 +33,5 @@
     <origin xyz="-0.07 -0.043 -0.0325" rpy="0 0 0"/>
     <geometry>
-      <mesh filename="file://$(find thunder_description)/meshes/front_wheel_left_1.stl" scale="0.001 0.001 0.001"/>
+      <mesh filename="file://$(find thunder_description)/meshes/front_wheel_left.stl" scale="0.001 0.001 0.001"/>
     </geometry>
     <material name="silver"/>
@@ -40,9 +40,9 @@
     <origin xyz="-0.07 -0.043 -0.0325" rpy="0 0 0"/>
     <geometry>
-      <mesh filename="file://$(find thunder_description)/meshes/front_wheel_left_1.stl" scale="0.001 0.001 0.001"/>
-    </geometry>
-  </collision>
-</link>
-<link name="front_wheel_right_1">
+      <mesh filename="file://$(find thunder_description)/meshes/front_wheel_left.stl" scale="0.001 0.001 0.001"/>
+    </geometry>
+  </collision>
+</link>
+<link name="front_wheel_right">
   <inertial>
     <origin xyz="0.0 -0.012500000000000004 0.0" rpy="0 0 0"/>
@@ -53,5 +53,5 @@
     <origin xyz="-0.07 0.043 -0.0325" rpy="0 0 0"/>
     <geometry>
-      <mesh filename="file://$(find thunder_description)/meshes/front_wheel_right_1.stl" scale="0.001 0.001 0.001"/>
+      <mesh filename="file://$(find thunder_description)/meshes/front_wheel_right.stl" scale="0.001 0.001 0.001"/>
     </geometry>
     <material name="silver"/>
@@ -60,9 +60,9 @@
     <origin xyz="-0.07 0.043 -0.0325" rpy="0 0 0"/>
     <geometry>
-      <mesh filename="file://$(find thunder_description)/meshes/front_wheel_right_1.stl" scale="0.001 0.001 0.001"/>
-    </geometry>
-  </collision>
-</link>
-<link name="rear_wheel_left_1">
+      <mesh filename="file://$(find thunder_description)/meshes/front_wheel_right.stl" scale="0.001 0.001 0.001"/>
+    </geometry>
+  </collision>
+</link>
+<link name="rear_wheel_left">
   <inertial>
     <origin xyz="2.7755575615628914e-17 0.012500000000000004 0.0" rpy="0 0 0"/>
@@ -73,5 +73,5 @@
     <origin xyz="0.07 -0.043 -0.0325" rpy="0 0 0"/>
     <geometry>
-      <mesh filename="file://$(find thunder_description)/meshes/rear_wheel_left_1.stl" scale="0.001 0.001 0.001"/>
+      <mesh filename="file://$(find thunder_description)/meshes/rear_wheel_left.stl" scale="0.001 0.001 0.001"/>
     </geometry>
     <material name="silver"/>
@@ -80,9 +80,9 @@
     <origin xyz="0.07 -0.043 -0.0325" rpy="0 0 0"/>
     <geometry>
-      <mesh filename="file://$(find thunder_description)/meshes/rear_wheel_left_1.stl" scale="0.001 0.001 0.001"/>
-    </geometry>
-  </collision>
-</link>
-<link name="rear_wheel_right_1">
+      <mesh filename="file://$(find thunder_description)/meshes/rear_wheel_left.stl" scale="0.001 0.001 0.001"/>
+    </geometry>
+  </collision>
+</link>
+<link name="rear_wheel_right">
   <inertial>
     <origin xyz="1.3877787807814457e-17 -0.012500000000000004 0.0" rpy="0 0 0"/>
@@ -93,5 +93,5 @@
     <origin xyz="0.07 0.043 -0.0325" rpy="0 0 0"/>
     <geometry>
-      <mesh filename="file://$(find thunder_description)/meshes/rear_wheel_right_1.stl" scale="0.001 0.001 0.001"/>
+      <mesh filename="file://$(find thunder_description)/meshes/rear_wheel_right.stl" scale="0.001 0.001 0.001"/>
     </geometry>
     <material name="silver"/>
@@ -100,9 +100,9 @@
     <origin xyz="0.07 0.043 -0.0325" rpy="0 0 0"/>
     <geometry>
-      <mesh filename="file://$(find thunder_description)/meshes/rear_wheel_right_1.stl" scale="0.001 0.001 0.001"/>
-    </geometry>
-  </collision>
-</link>
-<link name="lidar_1">
+      <mesh filename="file://$(find thunder_description)/meshes/rear_wheel_right.stl" scale="0.001 0.001 0.001"/>
+    </geometry>
+  </collision>
+</link>
+<link name="lidar">
   <inertial>
     <origin xyz="3.469446951953614e-18 0.0 0.010000000000000037" rpy="0 0 0"/>
@@ -113,5 +113,5 @@
     <origin xyz="0.015 -0.0 -0.1415" rpy="0 0 0"/>
     <geometry>
-      <mesh filename="file://$(find thunder_description)/meshes/lidar_1.stl" scale="0.001 0.001 0.001"/>
+      <mesh filename="file://$(find thunder_description)/meshes/lidar.stl" scale="0.001 0.001 0.001"/>
     </geometry>
     <material name="silver"/>
@@ -120,9 +120,9 @@
     <origin xyz="0.015 -0.0 -0.1415" rpy="0 0 0"/>
     <geometry>
-      <mesh filename="file://$(find thunder_description)/meshes/lidar_1.stl" scale="0.001 0.001 0.001"/>
-    </geometry>
-  </collision>
-</link>
-<link name="camera_1">
+      <mesh filename="file://$(find thunder_description)/meshes/lidar.stl" scale="0.001 0.001 0.001"/>
+    </geometry>
+  </collision>
+</link>
+<link name="camera">
   <inertial>
     <origin xyz="0.0 0.0 0.007500000000000007" rpy="0 0 0"/>
@@ -133,5 +133,5 @@
     <origin xyz="-0.095 -0.0 -0.1075" rpy="0 0 0"/>
     <geometry>
-      <mesh filename="file://$(find thunder_description)/meshes/camera_1.stl" scale="0.001 0.001 0.001"/>
+      <mesh filename="file://$(find thunder_description)/meshes/camera.stl" scale="0.001 0.001 0.001"/>
     </geometry>
     <material name="silver"/>
@@ -140,9 +140,9 @@
     <origin xyz="-0.095 -0.0 -0.1075" rpy="0 0 0"/>
     <geometry>
-      <mesh filename="file://$(find thunder_description)/meshes/camera_1.stl" scale="0.001 0.001 0.001"/>
-    </geometry>
-  </collision>
-</link>
-<link name="imu_1">
+      <mesh filename="file://$(find thunder_description)/meshes/camera.stl" scale="0.001 0.001 0.001"/>
+    </geometry>
+  </collision>
+</link>
+<link name="imu">
   <inertial>
     <origin xyz="0.0 0.0 0.0010000000000000009" rpy="0 0 0"/>
@@ -153,5 +153,5 @@
     <origin xyz="0.09 -0.0 -0.1075" rpy="0 0 0"/>
     <geometry>
-      <mesh filename="file://$(find thunder_description)/meshes/imu_1.stl" scale="0.001 0.001 0.001"/>
+      <mesh filename="file://$(find thunder_description)/meshes/imu.stl" scale="0.001 0.001 0.001"/>
     </geometry>
     <material name="silver"/>
@@ -160,5 +160,5 @@
     <origin xyz="0.09 -0.0 -0.1075" rpy="0 0 0"/>
     <geometry>
-      <mesh filename="file://$(find thunder_description)/meshes/imu_1.stl" scale="0.001 0.001 0.001"/>
+      <mesh filename="file://$(find thunder_description)/meshes/imu.stl" scale="0.001 0.001 0.001"/>
     </geometry>
   </collision>
@@ -167,5 +167,5 @@
   <origin xyz="0.07 0.043 0.0325" rpy="0 0 0"/>
   <parent link="base_link"/>
-  <child link="front_wheel_left_1"/>
+  <child link="front_wheel_left"/>
   <axis xyz="0.0 1.0 0.0"/>
 </joint>
@@ -173,5 +173,5 @@
   <origin xyz="0.07 -0.043 0.0325" rpy="0 0 0"/>
   <parent link="base_link"/>
-  <child link="front_wheel_right_1"/>
+  <child link="front_wheel_right"/>
   <axis xyz="0.0 -1.0 0.0"/>
 </joint>
@@ -179,5 +179,5 @@
   <origin xyz="-0.07 0.043 0.0325" rpy="0 0 0"/>
   <parent link="base_link"/>
-  <child link="rear_wheel_left_1"/>
+  <child link="rear_wheel_left"/>
   <axis xyz="0.0 1.0 0.0"/>
 </joint>
@@ -185,5 +185,5 @@
   <origin xyz="-0.07 -0.043 0.0325" rpy="0 0 0"/>
   <parent link="base_link"/>
-  <child link="rear_wheel_right_1"/>
+  <child link="rear_wheel_right"/>
   <axis xyz="0.0 -1.0 0.0"/>
 </joint>
@@ -191,15 +191,15 @@
   <origin xyz="-0.015 0.0 0.1415" rpy="0 0 0"/>
   <parent link="base_link"/>
-  <child link="lidar_1"/>
+  <child link="lidar"/>
 </joint>
 <joint name="camera_link" type="fixed">
   <origin xyz="0.095 0.0 0.1075" rpy="0 0 0"/>
   <parent link="base_link"/>
-  <child link="camera_1"/>
+  <child link="camera"/>
 </joint>
 <joint name="imu_link" type="fixed">
   <origin xyz="-0.09 0.0 0.1075" rpy="0 0 0"/>
   <parent link="base_link"/>
-  <child link="imu_1"/>
+  <child link="imu"/>
 </joint>
 </robot>

Commit message: fix: add dummy root_link to resolve KDL root inertia warning in Gazebo

File: thunder_description/urdf/thunder.xacro (robot description, xacro)
@@ -4,4 +4,5 @@
 <xacro:include filename="$(find thunder_description)/urdf/thunder.trans" />
 <xacro:include filename="$(find thunder_description)/urdf/thunder.gazebo" />
+<link name="root_link"/>
 <link name="base_link">
   <inertial>
@@ -164,4 +165,8 @@
   </collision>
 </link>
+<joint name="root_joint" type="fixed">
+  <parent link="root_link"/>
+  <child link="base_link"/>
+</joint>
 <joint name="front_wheel_left_joint" type="continuous">
   <origin xyz="0.07 0.043 0.0325" rpy="0 0 0"/>
